File: 01_Hardware/02_KiCad/air-quality-sensor/air-quality-sensor.kicad_sch (KiCad schematic)
At the start: 4 parts

Commit message: Finished layout of d70mm PCB
Parts:
- removed H2, H4: M2.5, MountingHole:MountingHole_2.5mm_Pad_Via, symbol Mechanical:MountingHole_Pad_MP
